File: pcb/power.kicad_sch (KiCad schematic)
At the start: 18 parts

Commit message: [temp]
Parts:
- added C? (x2): 100nF, symbol Device:C_Small
- added C?: 10nF, symbol Device:C_Small
- added C? (x2): 1uF, symbol Device:C_Small
- added C?: 10uF, symbol Device:C_Small
- added C? (x3): 22uF, symbol Device:C_Small
- added C?: 22nF, symbol Device:C_Small
- added L?: 2uH, symbol Device:L_Small
- added R?: 20K, symbol Device:R_Small
- added R?: 180K, symbol Device:R_Small
- added R?: 0R, symbol Device:R_Small
- added R?: 120K, symbol Device:R_Small
- added R?: 390K, symbol Device:R_Small
- added R?: 8K, symbol Device:R_Small
- added U?: MP2229, Package_DFN_QFN:MPS_QFN-14, symbol Regulator_Switching:MP2229
- added U?: TPS7A3001DRBx, Package_SON:Texas_S-PVSON-N8_1, symbol Regulator_Linear:TPS7A3001DRBx
Connections:
- net +6V: now also C?.1, C?.1, L?.2, R?.2
- net GND: now also C?.2, C?.2, C?.2, C?.2, C?.2, C?.2, C?.2, C?.2, C?.2, R?.1, R?.2, R?.2, U?.1 (GND), U?.12 (GND), U?.13 (GND), U?.14 (GND), U?.4 (GND), U?.5 (LPM), U?.9 (Pad)
- net at C?.1, U?.5 (-VOUT): now also C?.1, U?.5 (EN), U?.8 (IN)
- net +16V renamed IN
- net IN: now also C?.1, C?.1, U?.15 (IN), U?.3 (IN)
- new net: C?.1, U?.9 (VCC)
- new net: C?.1, U?.6 (NR/SS)
- new net: C?.2, L?.1, U?.11 (SW), U?.2 (SW)
- new net: R?.1, R?.2, R?.2
- new net: C?.1, U?.10 (BST)
- new net: R?.1, U?.6 (FB)
- new net: C?.1, U?.7 (SS)
- new net: R?.1, U?.8 (FREQ/SYNC)
- new net: R?.1, R?.2, U?.2 (FB)
- new net -5V: C?.1, R?.1, U?.1 (OUT)
- no-connect marks 3 -> 4
Other:
- note removed: "TPS7A3001 NEG LINEAR REGULATOR"
- company: (none) -> Nanjing wuyou electronic technology company
- title: (none) -> Power
- moved on the sheet: C?, R?, U?

Commit message: [feature] sch finish
Parts:
- gave numbers to parts that had none: 37
Connections:
- net GND: now also U9.3 (GND)

Commit message: [sch] finish footprint assignment
Parts:
- C18, C19, C20, C21, C22, C23, C26, C27, C28, C29, C30, C35, C36: footprint (none) -> Capacitor_SMD:C_0805_2012Metric
- C24, C25, C31, C32, C33, C34, C37: footprint (none) -> Capacitor_SMD:C_0603_1608Metric
- L1: footprint (none) -> Inductor_SMD:L_TDK_SLF7055
- R10, R11, R12, R13, R14, R5, R6, R7, R8, R9: footprint (none) -> Resistor_SMD:R_0603_1608Metric
- U9: footprint (none) -> Package_SO:SOIC-8_3.9x4.9mm_P1.27mm
Changed lines of the file:
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@@
       (effects (font (size 1.27 1.27)) (justify left))
     )
-    (property "Footprint" "" (id 2) (at 83.82 181.61 0)
+    (property "Footprint" "Capacitor_SMD:C_0805_2012Metric" (id 2) (at 83.82 181.61 0)
       (effects (font (size 1.27 1.27)) hide)
     )
@@
       (effects (font (size 1.27 1.27)) (justify left))
     )
-    (property "Footprint" "" (id 2) (at 58.42 68.58 0)
+    (property "Footprint" "Capacitor_SMD:C_0603_1608Metric" (id 2) (at 58.42 68.58 0)
       (effects (font (size 1.27 1.27)) hide)
     )
@@
       (effects (font (size 1.27 1.27)) (justify left))
     )
-    (property "Footprint" "" (id 2) (at 118.11 187.96 0)
+    (property "Footprint" "Capacitor_SMD:C_0603_1608Metric" (id 2) (at 118.11 187.96 0)
       (effects (font (size 1.27 1.27)) hide)
     )
@@
       (effects (font (size 1.27 1.27)) (justify left))
     )
-    (property "Footprint" "" (id 2) (at 88.9 29.21 0)
+    (property "Footprint" "Capacitor_SMD:C_0805_2012Metric" (id 2) (at 88.9 29.21 0)
       (effects (font (size 1.27 1.27)) hide)
     )
@@
     (property "Reference" "L1" (id 0) (at 111.76 59.69 90))
     (property "Value" "2uH" (id 1) (at 111.76 62.23 90))
-    (property "Footprint" "" (id 2) (at 111.76 64.77 0)
+    (property "Footprint" "Inductor_SMD:L_TDK_SLF7055" (id 2) (at 111.76 64.77 0)
       (effects (font (size 1.27 1.27)) hide)
     )
@@
       (effects (font (size 1.27 1.27)) (justify right))
     )
-    (property "Footprint" "" (id 2) (at 120.65 76.2 0)
+    (property "Footprint" "Resistor_SMD:R_0603_1608Metric" (id 2) (at 120.65 76.2 0)
       (effects (font (size 1.27 1.27)) hide)
     )
@@
       (effects (font (size 1.27 1.27)) (justify left))
     )
-    (property "Footprint" "" (id 2) (at 78.74 110.49 0)
+    (property "Footprint" "Resistor_SMD:R_0603_1608Metric" (id 2) (at 78.74 110.49 0)
       (effects (font (size 1.27 1.27)) hide)
     )
@@
       (effects (font (size 1.27 1.27)) (justify left))
     )
-    (property "Footprint" "" (id 2) (at 43.5314 107.95 0)
+    (property "Footprint" "Capacitor_SMD:C_0805_2012Metric" (id 2) (at 43.5314 107.95 0)
       (effects (font (size 1.27 1.27)) hide)
     )
@@
       (effects (font (size 1.27 1.27)) (justify left))
     )
-    (property "Footprint" "" (id 2) (at 165.1 181.61 0)
+    (property "Footprint" "Capacitor_SMD:C_0603_1608Metric" (id 2) (at 165.1 181.61 0)
       (effects (font (size 1.27 1.27)) hide)
     )
@@
       (effects (font (size 1.27 1.27)) (justify left))
     )
-    (property "Footprint" "" (id 2) (at 48.26 68.58 0)
+    (property "Footprint" "Capacitor_SMD:C_0805_2012Metric" (id 2) (at 48.26 68.58 0)
       (effects (font (size 1.27 1.27)) hide)
     )
@@
       (effects (font (size 1.27 1.27)) (justify right))
     )
-    (property "Footprint" "" (id 2) (at 120.65 68.58 0)
+    (property "Footprint" "Resistor_SMD:R_0603_1608Metric" (id 2) (at 120.65 68.58 0)
       (effects (font (size 1.27 1.27)) hide)
     )
@@
       (effects (font (size 1.27 1.27)) (justify left))
     )
-    (property "Footprint" "" (id 2) (at 43.18 29.21 0)
+    (property "Footprint" "Capacitor_SMD:C_0805_2012Metric" (id 2) (at 43.18 29.21 0)
       (effects (font (size 1.27 1.27)) hide)
     )
@@
       (effects (font (size 1.27 1.27)) (justify left))
     )
-    (property "Footprint" "" (id 2) (at 96.52 181.61 0)
+    (property "Footprint" "Capacitor_SMD:C_0805_2012Metric" (id 2) (at 96.52 181.61 0)
       (effects (font (size 1.27 1.27)) hide)
     )
@@
       (effects (font (size 1.27 1.27)) (justify left))
     )
-    (property "Footprint" "" (id 2) (at 43.5314 142.24 0)
+    (property "Footprint" "Capacitor_SMD:C_0805_2012Metric" (id 2) (at 43.5314 142.24 0)
       (effects (font (size 1.27 1.27)) hide)
     )
@@
       (effects (font (size 1.27 1.27)) (justify left))
     )
-    (property "Footprint" "" (id 2) (at 78.74 105.41 0)
+    (property "Footprint" "Resistor_SMD:R_0603_1608Metric" (id 2) (at 78.74 105.41 0)
       (effects (font (size 1.27 1.27)) hide)
     )
@@
       (effects (font (size 1.27 1.27)) (justify left))
     )
-    (property "Footprint" "" (id 2) (at 88.9 107.95 0)
+    (property "Footprint" "Capacitor_SMD:C_0805_2012Metric" (id 2) (at 88.9 107.95 0)
       (effects (font (size 1.27 1.27)) hide)
     )
@@
     (property "Reference" "R10" (id 0) (at 110.49 66.04 90))
     (property "Value" "0R" (id 1) (at 110.49 68.58 90))
-    (property "Footprint" "" (id 2) (at 110.49 72.39 0)
+    (property "Footprint" "Resistor_SMD:R_0603_1608Metric" (id 2) (at 110.49 72.39 0)
       (effects (font (size 1.27 1.27)) hide)
     )
@@
       (effects (font (size 1.27 1.27)) (justify left))
     )
-    (property "Footprint" "" (id 2) (at 100.33 60.96 0)
+    (property "Footprint" "Capacitor_SMD:C_0603_1608Metric" (id 2) (at 100.33 60.96 0)
       (effects (font (size 1.27 1.27)) hide)
     )
@@
       (effects (font (size 1.27 1.27)) (justify left))
     )
-    (property "Footprint" "" (id 2) (at 153.67 186.69 0)
+    (property "Footprint" "Resistor_SMD:R_0603_1608Metric" (id 2) (at 153.67 186.69 0)
       (effects (font (size 1.27 1.27)) hide)
     )
@@
       (effects (font (size 1.27 1.27)) (justify left))
     )
-    (property "Footprint" "" (id 2) (at 44.45 176.53 0)
+    (property "Footprint" "Capacitor_SMD:C_0805_2012Metric" (id 2) (at 44.45 176.53 0)
       (effects (font (size 1.27 1.27)) hide)
     )
@@
       (effects (font (size 1.27 1.27)) (justify left))
     )
-    (property "Footprint" "" (id 2) (at 78.74 31.75 0)
+    (property "Footprint" "Resistor_SMD:R_0603_1608Metric" (id 2) (at 78.74 31.75 0)
       (effects (font (size 1.27 1.27)) hide)
     )
@@
       (effects (font (size 1.27 1.27)) (justify left))
     )
-    (property "Footprint" "" (id 2) (at 153.67 175.26 0)
+    (property "Footprint" "Resistor_SMD:R_0603_1608Metric" (id 2) (at 153.67 175.26 0)
       (effects (font (size 1.27 1.27)) hide)
     )
@@
       (effects (font (size 1.27 1.27)) (justify left))
     )
-    (property "Footprint" "" (id 2) (at 78.74 142.24 0)
+    (property "Footprint" "Capacitor_SMD:C_0603_1608Metric" (id 2) (at 78.74 142.24 0)
       (effects (font (size 1.27 1.27)) hide)
     )
@@
     (property "Reference" "U9" (id 0) (at 68.58 163.83 0))
     (property "Value" "LT1054L" (id 1) (at 68.58 166.37 0))
-    (property "Footprint" "" (id 2) (at 71.12 181.61 0)
+    (property "Footprint" "Package_SO:SOIC-8_3.9x4.9mm_P1.27mm" (id 2) (at 71.12 181.61 0)
       (effects (font (size 1.27 1.27)) hide)
     )
@@
       (effects (font (size 1.27 1.27)) (justify left))
     )
-    (property "Footprint" "" (id 2) (at 38.1 68.58 0)
+    (property "Footprint" "Capacitor_SMD:C_0805_2012Metric" (id 2) (at 38.1 68.58 0)
       (effects (font (size 1.27 1.27)) hide)
     )
@@
       (effects (font (size 1.27 1.27)) (justify left))
     )
-    (property "Footprint" "" (id 2) (at 78.74 26.67 0)
+    (property "Footprint" "Resistor_SMD:R_0603_1608Metric" (id 2) (at 78.74 26.67 0)
       (effects (font (size 1.27 1.27)) hide)
     )
@@
       (effects (font (size 1.27 1.27)) (justify left))
     )
-    (property "Footprint" "" (id 2) (at 100.33 80.01 0)
+    (property "Footprint" "Capacitor_SMD:C_0603_1608Metric" (id 2) (at 100.33 80.01 0)
       (effects (font (size 1.27 1.27)) hide)
     )
@@
       (effects (font (size 1.27 1.27)) (justify left))
     )
-    (property "Footprint" "" (id 2) (at 68.58 81.28 0)
+    (property "Footprint" "Resistor_SMD:R_0603_1608Metric" (id 2) (at 68.58 81.28 0)
       (effects (font (size 1.27 1.27)) hide)
     )
@@
       (effects (font (size 1.27 1.27)) (justify left))
     )
-    (property "Footprint" "" (id 2) (at 139.7 72.39 0)
+    (property "Footprint" "Capacitor_SMD:C_0805_2012Metric" (id 2) (at 139.7 72.39 0)
       (effects (font (size 1.27 1.27)) hide)
     )
@@
       (effects (font (size 1.27 1.27)) (justify left))
     )
-    (property "Footprint" "" (id 2) (at 88.9 142.24 0)
+    (property "Footprint" "Capacitor_SMD:C_0805_2012Metric" (id 2) (at 88.9 142.24 0)
       (effects (font (size 1.27 1.27)) hide)
     )
@@
       (effects (font (size 1.27 1.27)) (justify left))
     )
-    (property "Footprint" "" (id 2) (at 111.76 181.61 0)
+    (property "Footprint" "Capacitor_SMD:C_0603_1608Metric" (id 2) (at 111.76 181.61 0)
       (effects (font (size 1.27 1.27)) hide)
     )
@@
       (effects (font (size 1.27 1.27)) (justify left))
     )
-    (property "Footprint" "" (id 2) (at 129.54 72.39 0)
-      (effects (font (size 1.27 1.27)) hide)
-    )
+    (property "Footprint" "Capacitor_SMD:C_0805_2012Metric" (id 2) (at 129.54 72.39 0)
+      (effects (font (size 1.27 1.27)) hide)
+    )
